Commit message: first commit

File: ur_description/urdf/inc/ur.transmissions.xacro (robot description, xacro)
@@ -6,9 +6,10 @@
           this location. Nor can they rely on the existence of the macro.
   -->
-  <xacro:macro name="ur_arm_transmission" params="prefix hw_interface">
+  <xacro:macro name="ur_arm_transmission" params="prefix"> <!--hw_interface"-->
     <transmission name="${prefix}shoulder_pan_trans">
       <type>transmission_interface/SimpleTransmission</type>
       <joint name="${prefix}shoulder_pan_joint">
-        <hardwareInterface>${hw_interface}</hardwareInterface>
+	<hardwareInterface>hardware_interface/VelocityJointInterface</hardwareInterface>
+        <!--hardwareInterface>${hw_interface}</hardwareInterface-->
       </joint>
       <actuator name="${prefix}shoulder_pan_motor">
@@ -19,5 +20,6 @@
       <type>transmission_interface/SimpleTransmission</type>
       <joint name="${prefix}shoulder_lift_joint">
-        <hardwareInterface>${hw_interface}</hardwareInterface>
+	<hardwareInterface>hardware_interface/VelocityJointInterface</hardwareInterface>
+        <!--hardwareInterface>${hw_interface}</hardwareInterface-->
       </joint>
       <actuator name="${prefix}shoulder_lift_motor">
@@ -28,5 +30,6 @@
       <type>transmission_interface/SimpleTransmission</type>
       <joint name="${prefix}elbow_joint">
-        <hardwareInterface>${hw_interface}</hardwareInterface>
+	<hardwareInterface>hardware_interface/VelocityJointInterface</hardwareInterface>
+        <!--hardwareInterface>${hw_interface}</hardwareInterface-->
       </joint>
       <actuator name="${prefix}elbow_motor">
@@ -37,5 +40,6 @@
       <type>transmission_interface/SimpleTransmission</type>
       <joint name="${prefix}wrist_1_joint">
-        <hardwareInterface>${hw_interface}</hardwareInterface>
+	<hardwareInterface>hardware_interface/VelocityJointInterface</hardwareInterface>
+        <!--hardwareInterface>${hw_interface}</hardwareInterface-->
       </joint>
       <actuator name="${prefix}wrist_1_motor">
@@ -46,5 +50,6 @@
       <type>transmission_interface/SimpleTransmission</type>
       <joint name="${prefix}wrist_2_joint">
-        <hardwareInterface>${hw_interface}</hardwareInterface>
+	<hardwareInterface>hardware_interface/VelocityJointInterface</hardwareInterface>
+        <!--hardwareInterface>${hw_interface}</hardwareInterface-->
       </joint>
       <actuator name="${prefix}wrist_2_motor">
@@ -55,5 +60,6 @@
       <type>transmission_interface/SimpleTransmission</type>
       <joint name="${prefix}wrist_3_joint">
-        <hardwareInterface>${hw_interface}</hardwareInterface>
+  	<hardwareInterface>hardware_interface/VelocityJointInterface</hardwareInterface>
+        <!--hardwareInterface>${hw_interface}</hardwareInterface-->
       </joint>
       <actuator name="${prefix}wrist_3_motor">

File: ur_description/urdf/inc/ur5_macro.xacro (robot description, xacro)
@@ -23,5 +23,5 @@
    physical_parameters_file:='$(find ur_description)/config/ur5/physical_parameters.yaml'
    visual_parameters_file:='$(find ur_description)/config/ur5/visual_parameters.yaml'
-   transmission_hw_interface:=hardware_interface/PositionJointInterface
+   transmission_hw_interface:=hardware_interface/VelocityJointInterface
    safety_limits:=false
    safety_pos_margin:=0.15

File: ur_description/urdf/inc/ur_macro.xacro (robot description, xacro)
@@ -50,9 +50,22 @@
     physical_parameters_file
     visual_parameters_file
-    transmission_hw_interface:=hardware_interface/PositionJointInterface
+    transmission_hw_interface:=hardware_interface/VelocityJointInterface
     safety_limits:=false
     safety_pos_margin:=0.15
     safety_k_position:=20"
   >
+  <xacro:property name="ur5_d1" value="0.089159" />
+  <xacro:property name="ur5_a2" value="-0.42500" />
+  <xacro:property name="ur5_a3" value="-0.39225" />
+  <xacro:property name="ur5_d4" value="0.10915" />
+  <xacro:property name="ur5_d5" value="0.09465" />
+  <xacro:property name="ur5_d6" value="0.0823" />
+  <!-- link lengths used in model -->
+  <xacro:property name="shoulder_height" value="${ur5_d1}" />
+  <xacro:property name="upper_arm_length" value="${-ur5_a2}" />
+  <xacro:property name="forearm_length" value="${-ur5_a3}" />
+  <xacro:property name="wrist_1_length" value="${ur5_d4 - elbow_offset - shoulder_offset}" />
+  <xacro:property name="wrist_2_length" value="${ur5_d5}" />
+  <xacro:property name="wrist_3_length" value="${ur5_d6}" />
     <!-- Load configuration data from the provided .yaml files -->
     <xacro:read_model_data

File: ur_description/urdf/ur.xacro (robot description, xacro)
@@ -13,5 +13,5 @@
          - hardware_interface/EffortJointInterface
    -->
-   <xacro:arg name="transmission_hw_interface" default="hardware_interface/PositionJointInterface"/>
+   <xacro:arg name="transmission_hw_interface" default="hardware_interface/VelocityJointInterface"/>
    <xacro:arg name="safety_limits" default="false"/>
    <xacro:arg name="safety_pos_margin" default="0.15"/>

File: ur_gazebo/urdf/ur.xacro (robot description, xacro)
@@ -38,5 +38,5 @@
           controller .yaml files in the 'config' directory.
   -->
-  <xacro:arg name="transmission_hw_interface" default="hardware_interface/PositionJointInterface"/>
+  <xacro:arg name="transmission_hw_interface" default="hardware_interface/VelocityJointInterface"/>
   <xacro:arg name="safety_limits" default="false"/>
   <xacro:arg name="safety_pos_margin" default="0.15"/>

File: ur_gazebo/urdf/ur_macro.xacro (robot description, xacro)
@@ -37,5 +37,5 @@
    physical_parameters_file
    visual_parameters_file
-   transmission_hw_interface:=hardware_interface/PositionJointInterface
+   transmission_hw_interface:=hardware_interface/VelocityJointInterface
    safety_limits:=false safety_pos_margin:=0.15 safety_k_position:=20"
   >
